File: GROUP_09.sch (EAGLE design)
At the start: 29 parts, among them J1 POWER_JACKPTH_LOCK, U1 +12v, U3 TCA9546ATSSOP16, U4 TMUX1208QNF

Commit message: Schematic V1.02
Parts:
- renumbered U$3 to CY8CKIT059-TARGET
Connections:
- net MUX_A0/1.4C renamed MUX_A1/1.4C
Changed lines of the file:
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@@
 <part name="U3" library="Group_09_Library" deviceset="TCA9546A" device="TSSOP16"/>
 <part name="U4" library="Group_09_Library" deviceset="TMUX1208" device="QNF"/>
-<part name="U$3" library="CY8KIT-059" deviceset="CY8CKIT-059_TARGET" device=""/>
+<part name="CY8CKIT059-TARGET" library="CY8KIT-059" deviceset="CY8CKIT-059_TARGET" device=""/>
 <part name="J1" library="SparkFun-Connectors" deviceset="POWER_JACK" device="PTH_LOCK"/>
 <part name="C2" library="SparkFun-Capacitors" deviceset="0.33UF/330NF" device="-0805-50V-10%" value="0.33µF"/>
@@
 <attribute name="VALUE" x="196.85" y="30.48" size="3.81" layer="96"/>
 </instance>
-<instance part="U$3" gate="G$1" x="111.76" y="124.46" smashed="yes" rot="R270"/>
+<instance part="CY8CKIT059-TARGET" gate="G$1" x="111.76" y="124.46" smashed="yes" rot="R270"/>
 <instance part="J1" gate="G$1" x="82.55" y="143.51" smashed="yes">
 <attribute name="VALUE" x="72.39" y="153.67" size="1.778" layer="96" font="vector"/>
@@
 </segment>
 <segment>
-<pinref part="U$3" gate="G$1" pin="VDDIO"/>
+<pinref part="CY8CKIT059-TARGET" gate="G$1" pin="VDDIO"/>
 <pinref part="SUPPLY7" gate="G$1" pin="5V"/>
 <wire x1="129.54" y1="101.6" x2="129.54" y2="110.49" width="0.1524" layer="91"/>
 </segment>
 <segment>
-<pinref part="U$3" gate="G$1" pin="VDD"/>
+<pinref part="CY8CKIT059-TARGET" gate="G$1" pin="VDD"/>
 <wire x1="93.98" y1="38.1" x2="83.82" y2="38.1" width="0.1524" layer="91"/>
 <pinref part="SUPPLY8" gate="G$1" pin="5V"/>
@@
 </segment>
 <segment>
-<pinref part="U$3" gate="G$1" pin="GND3"/>
+<pinref part="CY8CKIT059-TARGET" gate="G$1" pin="GND3"/>
 <pinref part="GND8" gate="1" pin="GND"/>
 <wire x1="129.54" y1="99.06" x2="175.26" y2="99.06" width="0.1524" layer="91"/>
@@
 </segment>
 <segment>
-<pinref part="U$3" gate="G$1" pin="GND1"/>
+<pinref part="CY8CKIT059-TARGET" gate="G$1" pin="GND1"/>
 <wire x1="93.98" y1="40.64" x2="90.17" y2="40.64" width="0.1524" layer="91"/>
 <pinref part="GND7" gate="1" pin="GND"/>
@@
 </segment>
 <segment>
-<pinref part="U$3" gate="G$1" pin="P_3.7"/>
+<pinref part="CY8CKIT059-TARGET" gate="G$1" pin="P_3.7"/>
 <label x="73.66" y="81.28" size="1.778" layer="95" rot="R180" xref="yes"/>
 <wire x1="93.98" y1="81.28" x2="73.66" y2="81.28" width="0.1524" layer="91"/>
@@
 </segment>
 <segment>
-<pinref part="U$3" gate="G$1" pin="P_15.0"/>
+<pinref part="CY8CKIT059-TARGET" gate="G$1" pin="P_15.0"/>
 <wire x1="93.98" y1="78.74" x2="90.17" y2="78.74" width="0.1524" layer="91"/>
 <label x="90.17" y="78.74" size="1.778" layer="95" rot="R180" xref="yes"/>
@@
 </segment>
 <segment>
-<pinref part="U$3" gate="G$1" pin="P_2.5"/>
+<pinref part="CY8CKIT059-TARGET" gate="G$1" pin="P_2.5"/>
 <wire x1="129.54" y1="50.8" x2="142.24" y2="50.8" width="0.1524" layer="91"/>
 <label x="142.24" y="50.8" size="1.778" layer="95" xref="yes"/>
@@
 </segment>
 <segment>
-<pinref part="U$3" gate="G$1" pin="P_2.6"/>
+<pinref part="CY8CKIT059-TARGET" gate="G$1" pin="P_2.6"/>
 <wire x1="129.54" y1="53.34" x2="130.81" y2="53.34" width="0.1524" layer="91"/>
 <label x="130.81" y="53.34" size="1.778" layer="95" xref="yes"/>
@@
 </segment>
 <segment>
-<pinref part="U$3" gate="G$1" pin="P_2.7"/>
+<pinref part="CY8CKIT059-TARGET" gate="G$1" pin="P_2.7"/>
 <wire x1="129.54" y1="55.88" x2="142.24" y2="55.88" width="0.1524" layer="91"/>
 <label x="142.24" y="55.88" size="1.778" layer="95" xref="yes"/>
@@
 </segment>
 <segment>
-<pinref part="U$3" gate="G$1" pin="P_12.1"/>
+<pinref part="CY8CKIT059-TARGET" gate="G$1" pin="P_12.1"/>
 <wire x1="129.54" y1="73.66" x2="149.86" y2="73.66" width="0.1524" layer="91"/>
 <label x="149.86" y="73.66" size="1.778" layer="95" xref="yes"/>
@@
 </segment>
 <segment>
-<pinref part="U$3" gate="G$1" pin="P_12.0"/>
+<pinref part="CY8CKIT059-TARGET" gate="G$1" pin="P_12.0"/>
 <wire x1="129.54" y1="76.2" x2="137.16" y2="76.2" width="0.1524" layer="91"/>
 <label x="137.16" y="76.2" size="1.778" layer="95" xref="yes"/>
@@
 <net name="N$6" class="0">
 <segment>
-<pinref part="U$3" gate="G$1" pin="P_3.0"/>
+<pinref part="CY8CKIT059-TARGET" gate="G$1" pin="P_3.0"/>
 <pinref part="D1" gate="G$1" pin="A"/>
 <wire x1="93.98" y1="99.06" x2="91.44" y2="99.06" width="0.1524" layer="91"/>
@@
 <net name="MUX_OUT/2.5C" class="0">
 <segment>
-<pinref part="U$3" gate="G$1" pin="P_1.4"/>
+<pinref part="CY8CKIT059-TARGET" gate="G$1" pin="P_1.4"/>
 <wire x1="129.54" y1="88.9" x2="149.86" y2="88.9" width="0.1524" layer="91"/>
 <label x="149.86" y="88.9" size="1.778" layer="95" xref="yes"/>
@@
 <net name="MUX_A2/2.3C" class="0">
 <segment>
-<pinref part="U$3" gate="G$1" pin="P_1.5"/>
+<pinref part="CY8CKIT059-TARGET" gate="G$1" pin="P_1.5"/>
 <wire x1="129.54" y1="91.44" x2="130.81" y2="91.44" width="0.1524" layer="91"/>
 <label x="130.81" y="91.44" size="1.778" layer="95" xref="yes"/>
@@
 <net name="MUX_A1/2.3C" class="0">
 <segment>
-<pinref part="U$3" gate="G$1" pin="P_1.6"/>
+<pinref part="CY8CKIT059-TARGET" gate="G$1" pin="P_1.6"/>
 <wire x1="129.54" y1="93.98" x2="149.86" y2="93.98" width="0.1524" layer="91"/>
 <label x="149.86" y="93.98" size="1.778" layer="95" xref="yes"/>
@@
 <net name="MUX_A0/2.3C" class="0">
 <segment>
-<pinref part="U$3" gate="G$1" pin="P_1.7"/>
+<pinref part="CY8CKIT059-TARGET" gate="G$1" pin="P_1.7"/>
 <wire x1="129.54" y1="96.52" x2="130.81" y2="96.52" width="0.1524" layer="91"/>
 <label x="130.81" y="96.52" size="1.778" layer="95" xref="yes"/>
@@
 </segment>
 </net>
-<net name="MUX_A0/1.4C" class="0">
+<net name="MUX_A1/1.4C" class="0">
 <segment>
 <pinref part="U4" gate="A" pin="A1"/>
@@
 <segment>
 <pinref part="J6" gate="G$1" pin="1"/>
-<pinref part="U$3" gate="G$1" pin="P_0.5"/>
+<pinref part="CY8CKIT059-TARGET" gate="G$1" pin="P_0.5"/>
 <wire x1="87.63" y1="50.8" x2="93.98" y2="50.8" width="0.1524" layer="91"/>
 </segment>
@@
 <segment>
 <pinref part="J6" gate="G$1" pin="2"/>
-<pinref part="U$3" gate="G$1" pin="P_0.4"/>
+<pinref part="CY8CKIT059-TARGET" gate="G$1" pin="P_0.4"/>
 <wire x1="87.63" y1="53.34" x2="93.98" y2="53.34" width="0.1524" layer="91"/>
 </segment>
@@
 <segment>
 <pinref part="J6" gate="G$1" pin="3"/>
-<pinref part="U$3" gate="G$1" pin="P_0.3"/>
+<pinref part="CY8CKIT059-TARGET" gate="G$1" pin="P_0.3"/>
 <wire x1="87.63" y1="55.88" x2="93.98" y2="55.88" width="0.1524" layer="91"/>
 </segment>
@@
 <segment>
 <pinref part="J6" gate="G$1" pin="4"/>
-<pinref part="U$3" gate="G$1" pin="P_0.2"/>
+<pinref part="CY8CKIT059-TARGET" gate="G$1" pin="P_0.2"/>
 <wire x1="87.63" y1="58.42" x2="93.98" y2="58.42" width="0.1524" layer="91"/>
 </segment>
@@
 <segment>
 <pinref part="J6" gate="G$1" pin="5"/>
-<pinref part="U$3" gate="G$1" pin="P_0.1"/>
+<pinref part="CY8CKIT059-TARGET" gate="G$1" pin="P_0.1"/>
 <wire x1="87.63" y1="60.96" x2="93.98" y2="60.96" width="0.1524" layer="91"/>
 </segment>
@@
 <segment>
 <pinref part="J6" gate="G$1" pin="6"/>
-<pinref part="U$3" gate="G$1" pin="P_0.0"/>
+<pinref part="CY8CKIT059-TARGET" gate="G$1" pin="P_0.0"/>
 <wire x1="87.63" y1="63.5" x2="93.98" y2="63.5" width="0.1524" layer="91"/>
 </segment>

Commit message: Final version
Parts:
- J2, J3, J4, J5, J6, J7, J8, S1, U2: value (none) -> (none)
Connections:
- net N$12 renamed MIC_0.5
- net N$13 renamed MIC_0.4
- net N$14 renamed MIC_0.3
- net N$15 renamed MIC_0.2
- net N$16 renamed MIC_0.1
- net N$17 renamed MIC_0.0
- net N$18 renamed MUX_S8
- net N$19 renamed MUX_S7
- net N$20 renamed MUX_S6
- net N$21 renamed MUX_S5
- net N$22 renamed MUX_S4
- net N$23 renamed MUX_S3
- net N$24 renamed MUX_S2
- net N$25 renamed MUX_S1
- removed net MUX_A0/1.3C: U4.A0
- removed net MUX_A0/2.3C: CY8CKIT059-TARGET.P_1.7
- removed net MUX_A1/1.4C: U4.A1
- removed net MUX_A1/2.3C: CY8CKIT059-TARGET.P_1.6
- removed net MUX_A2/1.4C: U4.A2
- removed net MUX_A2/2.3C: CY8CKIT059-TARGET.P_1.5
- removed net MUX_OUT/1.4C: U4.D
- removed net MUX_OUT/2.5C: CY8CKIT059-TARGET.P_1.4
- removed net N$1: R2.2, U3.SD0
- removed net N$10: R6.1, U3.SD2
- removed net N$3: R3.2, U3.SC0
- removed net N$4: R4.2, U3.SD1
- removed net N$5: R5.2, U3.SC1
- removed net N$7: R9.1, U3.SC3
- removed net N$8: R8.1, U3.SD3
- removed net N$9: R7.1, U3.SC2
- new net MUX_A0: CY8CKIT059-TARGET.P_1.7, U4.A0
- new net MUX_A1: CY8CKIT059-TARGET.P_1.6, U4.A1
- new net MUX_A2: CY8CKIT059-TARGET.P_1.5, U4.A2
- new net MUX_OUT: CY8CKIT059-TARGET.P_1.4, U4.D
- net I2C_SCL_0: now also R3.2, U3.SC0
- net I2C_SCL_1: now also R5.2, U3.SC1
- net I2C_SCL_2: now also R7.1, U3.SC2
- net I2C_SCL_3: now also R9.1, U3.SC3
- net I2C_SDA_0: now also R2.2, U3.SD0
- net I2C_SDA_1: now also R4.2, U3.SD1
- net I2C_SDA_2: now also R6.1, U3.SD2
- net I2C_SDA_3: now also R8.1, U3.SD3
Other:
- note added: "HEADERS"
- note added: "I2C"
- note added: "MICRO"
- note added: "MUX"
- note added: "SENSORS"
- note added: "SUPPLY"
- moved on the sheet: C1, C2, C3, D1, J1, J2, J3, J4, J5, J6, J7, J8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
